Commit message: adjust reward for rj45

File: source/isaaclab_assets/isaaclab_assets/custom_assets/robots/lbr_description/urdf/kuka_blue/kuka_blue_rj45.urdf (robot description, URDF)
Before this commit: robot iiwa7, 12 links, 11 joints
Links:
- removed link link_lid
- added link link_rj45, mass 0.01; visual mesh filename=/home/blacktower27/code/python_code/CAM/IsaacLab/source/isa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 scale=1 1 1
Joints:
- removed joint joint_lid
- added joint joint_rj45: type fixed, parent link_tcp, child link_rj45, origin xyz=0.01 0.008 0.050 rpy=3.14159 0 0

Commit message: replace model for rj45 and fix the offset bugs

File: source/isaaclab_assets/isaaclab_assets/custom_assets/robots/lbr_description/urdf/kuka_blue/kuka_blue_rj45.urdf (robot description, URDF)
Before this commit: robot iiwa7, 12 links, 11 joints
Links:
- link link_rj45: geometry visual mesh filename=../../../../rj45/medium/rs_male_rj45.usd scale=1 1 1
Joints:
- joint joint_rj45: origin xyz=0.01 0.008 0.050 rpy=3.14159 0 0 -> xyz=0.0 0.0 0.0 rpy=3.14159 0 0
