Commit message: extend training, closer the init point

File: source/isaaclab_assets/isaaclab_assets/custom_assets/robots/lbr_description/urdf/kuka_blue/kuka_blue_bnc_small.urdf (robot description, URDF)
Before this commit: robot iiwa7, 12 links, 11 joints
Links:
- added link force_sensor
Joints:
- added joint joint_force_sensor: type fixed, parent link_7, child force_sensor, origin xyz=0 0 0.192 rpy=0 0 3.14
- joint joint_ee: origin xyz=0 0 0.035 rpy=0 0 3.14 -> xyz=0 0 0.035 rpy=0 0 0

File: source/isaaclab_assets/isaaclab_assets/custom_assets/robots/lbr_description/urdf/kuka_blue/kuka_blue_lid.urdf (robot description, URDF)
Before this commit: robot iiwa7, 12 links, 11 joints
Links:
- added link link_lid, mass 0.02; visual mesh filename=../../../../box/middle/Lid_Yellow.usd scale=1 1 1
- link force_sensor: geometry 
Joints:
- added joint joint_lid: type fixed, parent link_tcp, child link_lid, origin xyz=-0.0094 0.002 0.035 rpy=-2.5307 0 -1.5708

File: source/isaaclab_assets/isaaclab_assets/custom_assets/robots/lbr_description/urdf/kuka_blue/kuka_blue_rj45.urdf (robot description, URDF)
Before this commit: robot iiwa7, 12 links, 11 joints
Links:
- added link force_sensor
Joints:
- added joint joint_force_sensor: type fixed, parent link_7, child force_sensor, origin xyz=0 0 0.192 rpy=0 0 3.14
- joint joint_ee: origin xyz=0 0 0.035 rpy=0 0 3.14 -> xyz=0 0 0.035 rpy=0 0 0
