Commit message: adjust ee of kuka, settle init state

File: source/isaaclab_assets/isaaclab_assets/custom_assets/robots/lbr_description/urdf/kuka_blue/kuka_blue.urdf (robot description, URDF)
Before this commit: robot iiwa7, 11 links, 10 joints
Joints:
- joint joint_tcp: origin xyz=0.00243 0.0003 0.22498 rpy=0 0 0 -> xyz=0.00243 0.0003 0.3325 rpy=0 0 1.5708
- joint world_joint: origin xyz=0.5754642 -0.4159573 -0.2417773 rpy=0.0 0.0 0.0 -> xyz=0.0 0.0 0.0 rpy=0.0 0.0 0.0

Commit message: fix the collision, extend the horizon_length

File: source/isaaclab_assets/isaaclab_assets/custom_assets/robots/lbr_description/urdf/kuka_blue/kuka_blue.urdf (robot description, URDF)
Before this commit: robot iiwa7, 11 links, 10 joints
Links:
- added link link_lid, mass 0.02; collision mesh filename=/home/blacktower27/code/python_code/CAM/IsaacLab/source/isa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 scale=1 1 1; visual mesh filename=/home/blacktower27/code/python_code/CAM/IsaacLab/source/isa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 scale=1 1 1
Joints:
- added joint joint_lid: type fixed, parent link_tcp, child link_lid, origin xyz=-0.0094 0.002 0.035 rpy=-2.5307 0 -1.5708

Commit message: insert lid in box now working on kuka

File: source/isaaclab_assets/isaaclab_assets/custom_assets/robots/lbr_description/urdf/kuka_blue/kuka_blue.urdf (robot description, URDF)
Before this commit: robot iiwa7, 12 links, 11 joints
Links:
- link link_lid: geometry visual mesh filename=/home/blacktower27/code/python_code/CAM/IsaacLab/source/isa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 scale=1 1 1

Commit message: fix bug

File: source/isaaclab_assets/isaaclab_assets/custom_assets/robots/lbr_description/urdf/kuka_blue/kuka_blue.urdf (robot description, URDF)
Before this commit: robot iiwa7, 12 links, 11 joints
Links:
- link link_0: geometry collision mesh filename=../../meshes/iiwa7/collision/link_0.stl; visual mesh filename=../../meshes/iiwa7/visual/link_0.dae
- link link_1: geometry collision mesh filename=../../meshes/iiwa7/collision/link_1.stl; visual mesh filename=../../meshes/iiwa7/visual/link_1.dae
- link link_2: geometry collision mesh filename=../../meshes/iiwa7/collision/link_2.stl; visual mesh filename=../../meshes/iiwa7/visual/link_2.dae
- link link_3: geometry collision mesh filename=../../meshes/iiwa7/collision/link_3.stl; visual mesh filename=../../meshes/iiwa7/visual/link_3.dae
- link link_4: geometry collision mesh filename=../../meshes/iiwa7/collision/link_4.stl; visual mesh filename=../../meshes/iiwa7/visual/link_4.dae
- link link_5: geometry collision mesh filename=../../meshes/iiwa7/collision/link_5.stl; visual mesh filename=../../meshes/iiwa7/visual/link_5.dae
- link link_6: geometry collision mesh filename=../../meshes/iiwa7/collision/link_6.stl; visual mesh filename=../../meshes/iiwa7/visual/link_6.dae
- link link_7: geometry collision mesh filename=../../meshes/iiwa7/collision/link_7.stl; visual mesh filename=../../meshes/iiwa7/visual/link_7.dae
- link link_ee: geometry collision mesh filename=../../meshes/iiwa7/collision/aniket_gripper.stl scale=0.001 0.001 0.001; visual mesh filename=../../meshes/iiwa7/visual/aniket_gripper.obj scale=0.001 0.001 0.001
- link link_lid: geometry visual mesh filename=../../../../box/middle/Lid_Yellow.usd scale=1 1 1

File: source/isaaclab_assets/isaaclab_assets/custom_assets/robots/lbr_description/urdf/kuka_blue/kuka_blue_bnc_small.urdf (robot description, URDF)
Before this commit: robot iiwa7, 12 links, 11 joints
Links:
- link link_0: geometry collision mesh filename=../../meshes/iiwa7/collision/link_0.stl; visual mesh filename=../../meshes/iiwa7/visual/link_0.dae
- link link_1: geometry collision mesh filename=../../meshes/iiwa7/collision/link_1.stl; visual mesh filename=../../meshes/iiwa7/visual/link_1.dae
- link link_2: geometry collision mesh filename=../../meshes/iiwa7/collision/link_2.stl; visual mesh filename=../../meshes/iiwa7/visual/link_2.dae
- link link_3: geometry collision mesh filename=../../meshes/iiwa7/collision/link_3.stl; visual mesh filename=../../meshes/iiwa7/visual/link_3.dae
- link link_4: geometry collision mesh filename=../../meshes/iiwa7/collision/link_4.stl; visual mesh filename=../../meshes/iiwa7/visual/link_4.dae
- link link_5: geometry collision mesh filename=../../meshes/iiwa7/collision/link_5.stl; visual mesh filename=../../meshes/iiwa7/visual/link_5.dae
- link link_6: geometry collision mesh filename=../../meshes/iiwa7/collision/link_6.stl; visual mesh filename=../../meshes/iiwa7/visual/link_6.dae
- link link_7: geometry collision mesh filename=../../meshes/iiwa7/collision/link_7.stl; visual mesh filename=../../meshes/iiwa7/visual/link_7.dae
- link link_bnc: geometry visual mesh filename=../../../../bnc/small/Adi_BNC_Simulation_Small_Male.usd scale=1 1 1
- link link_ee: geometry collision mesh filename=../../meshes/iiwa7/collision/aniket_gripper.stl scale=0.001 0.001 0.001; visual mesh filename=../../meshes/iiwa7/visual/aniket_gripper.obj scale=0.001 0.001 0.001

File: source/isaaclab_assets/isaaclab_assets/custom_assets/robots/lbr_description/urdf/kuka_blue/kuka_blue_rj45.urdf (robot description, URDF)
Before this commit: robot iiwa7, 12 links, 11 joints
Links:
- link link_0: geometry collision mesh filename=../../meshes/iiwa7/collision/link_0.stl; visual mesh filename=../../meshes/iiwa7/visual/link_0.dae
- link link_1: geometry collision mesh filename=../../meshes/iiwa7/collision/link_1.stl; visual mesh filename=../../meshes/iiwa7/visual/link_1.dae
- link link_2: geometry collision mesh filename=../../meshes/iiwa7/collision/link_2.stl; visual mesh filename=../../meshes/iiwa7/visual/link_2.dae
- link link_3: geometry collision mesh filename=../../meshes/iiwa7/collision/link_3.stl; visual mesh filename=../../meshes/iiwa7/visual/link_3.dae
- link link_4: geometry collision mesh filename=../../meshes/iiwa7/collision/link_4.stl; visual mesh filename=../../meshes/iiwa7/visual/link_4.dae
- link link_5: geometry collision mesh filename=../../meshes/iiwa7/collision/link_5.stl; visual mesh filename=../../meshes/iiwa7/visual/link_5.dae
- link link_6: geometry collision mesh filename=../../meshes/iiwa7/collision/link_6.stl; visual mesh filename=../../meshes/iiwa7/visual/link_6.dae
- link link_7: geometry collision mesh filename=../../meshes/iiwa7/collision/link_7.stl; visual mesh filename=../../meshes/iiwa7/visual/link_7.dae
- link link_ee: geometry collision mesh filename=../../meshes/iiwa7/collision/aniket_gripper.stl scale=0.001 0.001 0.001; visual mesh filename=../../meshes/iiwa7/visual/aniket_gripper.obj scale=0.001 0.001 0.001
- link link_rj45: geometry visual mesh filename=../../../../rj45/medium/Adi_Medium_RJ45_Male_Raw_Colored.usd scale=1 1 1

Commit message: fix the bug of settle the arm

File: source/isaaclab_assets/isaaclab_assets/custom_assets/robots/lbr_description/urdf/kuka_blue/kuka_blue.urdf (robot description, URDF)
Before this commit: robot iiwa7, 12 links, 11 joints
Links:
- removed link world
- link link_tcp: geometry visual cylinder length=0.04 radius=0.0025; visual sphere radius=0.012
Joints:
- removed joint world_joint

File: source/isaaclab_assets/isaaclab_assets/custom_assets/robots/lbr_description/urdf/kuka_blue/kuka_blue.xacro (robot description, xacro)
@@ -50,5 +50,25 @@
     </joint>
     <!-- TCP Link -->
-    <link name="link_tcp"/>
+    <link name="link_tcp">
+        <!-- Visual-only TCP marker: sphere marks the exact frame origin; cylinder shows local +Z. -->
+        <visual>
+            <origin rpy="0 0 0" xyz="0 0 0"/>
+            <geometry>
+                <sphere radius="0.012"/>
+            </geometry>
+            <material name="tcp_marker_yellow">
+                <color rgba="1 0.85 0.1 1"/>
+            </material>
+        </visual>
+        <visual>
+            <origin rpy="0 0 0" xyz="0 0 0.02"/>
+            <geometry>
+                <cylinder length="0.04" radius="0.0025"/>
+            </geometry>
+            <material name="tcp_marker_cyan">
+                <color rgba="0.1 0.9 1 1"/>
+            </material>
+        </visual>
+    </link>
     <joint name="joint_tcp" type="fixed">
         <parent link="link_ee"/>

File: source/isaaclab_assets/isaaclab_assets/custom_assets/robots/lbr_description/urdf/kuka_blue/kuka_blue_bnc_small.urdf (robot description, URDF)
Before this commit: robot iiwa7, 13 links, 12 joints
Links:
- removed link world
- link link_bnc: geometry visual mesh filename=../../../../bnc/small/Adi_BNC_Simulation_Small_Male.stl scale=0.001 0.001 0.001
- link link_tcp: geometry visual cylinder length=0.04 radius=0.0025; visual sphere radius=0.012
Joints:
- removed joint world_joint

File: source/isaaclab_assets/isaaclab_assets/custom_assets/robots/lbr_description/urdf/kuka_blue/kuka_blue_lid.urdf (robot description, URDF)
Before this commit: robot iiwa7, 13 links, 12 joints
Links:
- removed link world
- link link_tcp: geometry visual cylinder length=0.04 radius=0.0025; visual sphere radius=0.012
Joints:
- removed joint world_joint

File: source/isaaclab_assets/isaaclab_assets/custom_assets/robots/lbr_description/urdf/kuka_blue/kuka_blue_rj45.urdf (robot description, URDF)
Before this commit: robot iiwa7, 13 links, 12 joints
Links:
- removed link world
- link link_tcp: geometry visual cylinder length=0.04 radius=0.0025; visual sphere radius=0.012
Joints:
- removed joint world_joint
